Commit message: add new urdf wbc improper

File: resource/demir_1/demir_1.urdf (robot description, URDF)
Before this commit: robot opy_v05, 18 links, 17 joints
Links:
- removed link opy_v05/abad_1
- removed link opy_v05/abad_2
- removed link opy_v05/abad_3
- removed link opy_v05/abad_4
- removed link opy_v05/base_link
- removed link opy_v05/base_link_inertia
- removed link opy_v05/foot_1
- removed link opy_v05/foot_2
- removed link opy_v05/foot_3
- removed link opy_v05/foot_4
- removed link opy_v05/hip_1
- removed link opy_v05/hip_2
- removed link opy_v05/hip_3
- removed link opy_v05/hip_4
- removed link opy_v05/knee_1
- removed link opy_v05/knee_2
- removed link opy_v05/knee_3
- removed link opy_v05/knee_4
- added link demir_1/abad_1, mass 1.2834; collision mesh filename=package://opy-highlevel/meshes/demir_1/ABDUCTION.stl; visual mesh filename=package://opy-highlevel/meshes/demir_1/ABDUCTION_1.stl
- added link demir_1/abad_2, mass 1.2834; collision mesh filename=package://opy-highlevel/meshes/demir_1/ABDUCTION.stl; visual mesh filename=package://opy-highlevel/meshes/demir_1/ABDUCTION_2.stl
- added link demir_1/abad_3, mass 1.2834; collision mesh filename=package://opy-highlevel/meshes/demir_1/ABDUCTION.stl; visual mesh filename=package://opy-highlevel/meshes/demir_1/ABDUCTION_3.stl
- added link demir_1/abad_4, mass 1.2834; collision mesh filename=package://opy-highlevel/meshes/demir_1/ABDUCTION.stl; visual mesh filename=package://opy-highlevel/meshes/demir_1/ABDUCTION_4.stl
- added link demir_1/base_link
- added link demir_1/base_link_inertia, mass 14.2; collision mesh filename=package://opy-highlevel/meshes/demir_1/GOVDE.stl; visual mesh filename=package://opy-highlevel/meshes/demir_1/GOVDE.stl
- added link demir_1/foot_1, mass 0.1737; collision sphere radius=0.02; visual mesh filename=package://opy-highlevel/meshes/demir_1/FOOT.stl
- added link demir_1/foot_2, mass 0.1737; collision sphere radius=0.02; visual mesh filename=package://opy-highlevel/meshes/demir_1/FOOT.stl
- added link demir_1/foot_3, mass 0.1737; collision sphere radius=0.02; visual mesh filename=package://opy-highlevel/meshes/demir_1/FOOT.stl
- added link demir_1/foot_4, mass 0.1737; collision sphere radius=0.02; visual mesh filename=package://opy-highlevel/meshes/demir_1/FOOT.stl
- added link demir_1/hip_1, mass 2.3239; collision mesh filename=package://opy-highlevel/meshes/demir_1/HIP_R.stl; visual mesh filename=package://opy-highlevel/meshes/demir_1/HIP_R.stl
- added link demir_1/hip_2, mass 2.3239; collision mesh filename=package://opy-highlevel/meshes/demir_1/HIP_L.stl; visual mesh filename=package://opy-highlevel/meshes/demir_1/HIP_L.stl
- added link demir_1/hip_3, mass 2.3239; collision mesh filename=package://opy-highlevel/meshes/demir_1/HIP_R.stl; visual mesh filename=package://opy-highlevel/meshes/demir_1/HIP_R.stl
- added link demir_1/hip_4, mass 2.3239; collision mesh filename=package://opy-highlevel/meshes/demir_1/HIP_L.stl; visual mesh filename=package://opy-highlevel/meshes/demir_1/HIP_L.stl
- added link demir_1/knee_1, mass 0.3966; collision mesh filename=package://opy-highlevel/meshes/demir_1/KNEE.stl; visual mesh filename=package://opy-highlevel/meshes/demir_1/KNEE.stl
- added link demir_1/knee_2, mass 0.3966; collision mesh filename=package://opy-highlevel/meshes/demir_1/KNEE.stl; visual mesh filename=package://opy-highlevel/meshes/demir_1/KNEE.stl
- added link demir_1/knee_3, mass 0.3966; collision mesh filename=package://opy-highlevel/meshes/demir_1/KNEE.stl; visual mesh filename=package://opy-highlevel/meshes/demir_1/KNEE.stl
- added link demir_1/knee_4, mass 0.3966; collision mesh filename=package://opy-highlevel/meshes/demir_1/KNEE.stl; visual mesh filename=package://opy-highlevel/meshes/demir_1/KNEE.stl
Joints:
- removed joint opy_v05/abad_1_joint
- removed joint opy_v05/abad_2_joint
- removed joint opy_v05/abad_3_joint
- removed joint opy_v05/abad_4_joint
- removed joint opy_v05/base_joint
- removed joint opy_v05/foot_1_joint
- removed joint opy_v05/foot_2_joint
- removed joint opy_v05/foot_3_joint
- removed joint opy_v05/foot_4_joint
- removed joint opy_v05/hip_1_joint
- removed joint opy_v05/hip_2_joint
- removed joint opy_v05/hip_3_joint
- removed joint opy_v05/hip_4_joint
- removed joint opy_v05/knee_1_joint
- removed joint opy_v05/knee_2_joint
- removed joint opy_v05/knee_3_joint
- removed joint opy_v05/knee_4_joint
- added joint demir_1/abad_1_joint: type revolute, parent demir_1/base_link, child demir_1/abad_1, origin xyz=0.2238953 -0.0655252 0 rpy=0 0 0, axis 1 0 0, limit lower=-3.141592653589793 upper=3.141592653589793 effort=1e3 velocity=1e3
- added joint demir_1/abad_2_joint: type revolute, parent demir_1/base_link, child demir_1/abad_2, origin xyz=0.2238953 0.0655252 0 rpy=0 0 0, axis 1 0 0, limit lower=-3.141592653589793 upper=3.141592653589793 effort=1e3 velocity=1e3
- added joint demir_1/abad_3_joint: type revolute, parent demir_1/base_link, child demir_1/abad_3, origin xyz=-0.2238953 -0.0655252 0 rpy=0 0 0, axis 1 0 0, limit lower=-3.141592653589793 upper=3.141592653589793 effort=1e3 velocity=1e3
- added joint demir_1/abad_4_joint: type revolute, parent demir_1/base_link, child demir_1/abad_4, origin xyz=-0.2238953 0.0655252 0 rpy=0 0 0, axis 1 0 0, limit lower=-3.141592653589793 upper=3.141592653589793 effort=1e3 velocity=1e3
- added joint demir_1/base_joint: type revolute, parent demir_1/base_link, child demir_1/base_link_inertia, origin xyz=0 0 0 rpy=0 0 0
- added joint demir_1/foot_1_joint: type fixed, parent demir_1/knee_1, child demir_1/foot_1, origin xyz=0.0 -0.0 -0.2883978 rpy=0 0 0
- added joint demir_1/foot_2_joint: type fixed, parent demir_1/knee_2, child demir_1/foot_2, origin xyz=0.0 0.0 -0.2883978 rpy=0 0 0
- added joint demir_1/foot_3_joint: type fixed, parent demir_1/knee_3, child demir_1/foot_3, origin xyz=0.0 -0.0 -0.2883978 rpy=0 0 0
- added joint demir_1/foot_4_joint: type fixed, parent demir_1/knee_4, child demir_1/foot_4, origin xyz=0.0 0.0 -0.2883978 rpy=0 0 0
- added joint demir_1/hip_1_joint: type revolute, parent demir_1/abad_1, child demir_1/hip_1, origin xyz=0.0644992 -0.025 0 rpy=0 0 3.14, axis 0 1 0, limit lower=-3.141592653589793 upper=3.141592653589793 effort=1e3 velocity=1e3
- added joint demir_1/hip_2_joint: type revolute, parent demir_1/abad_2, child demir_1/hip_2, origin xyz=0.0644992 0.025 0 rpy=0 0 3.14, axis 0 1 0, limit lower=-3.141592653589793 upper=3.141592653589793 effort=1e3 velocity=1e3
- added joint demir_1/hip_3_joint: type revolute, parent demir_1/abad_3, child demir_1/hip_3, origin xyz=-0.0644992 -0.025 0 rpy=0 0 3.14, axis 0 1 0, limit lower=-3.141592653589793 upper=3.141592653589793 effort=1e3 velocity=1e3
- added joint demir_1/hip_4_joint: type revolute, parent demir_1/abad_4, child demir_1/hip_4, origin xyz=-0.0644992 0.025 0 rpy=0 0 3.14, axis 0 1 0, limit lower=-3.141592653589793 upper=3.141592653589793 effort=1e3 velocity=1e3
- added joint demir_1/knee_1_joint: type revolute, parent demir_1/hip_1, child demir_1/knee_1, origin xyz=0.0 0.07885 -0.27 rpy=0 0 0, axis 0 1 0, limit lower=-3.141592653589793 upper=3.141592653589793 effort=1e3 velocity=1e3
- added joint demir_1/knee_2_joint: type revolute, parent demir_1/hip_2, child demir_1/knee_2, origin xyz=0.0 -0.07885 -0.27 rpy=0 0 0, axis 0 1 0, limit lower=-3.141592653589793 upper=3.141592653589793 effort=1e3 velocity=1e3
- added joint demir_1/knee_3_joint: type revolute, parent demir_1/hip_3, child demir_1/knee_3, origin xyz=0.0 0.07885 -0.27 rpy=0 0 0, axis 0 1 0, limit lower=-3.141592653589793 upper=3.141592653589793 effort=1e3 velocity=1e3
- added joint demir_1/knee_4_joint: type revolute, parent demir_1/hip_4, child demir_1/knee_4, origin xyz=0.0 -0.07885 -0.27 rpy=0 0 0, axis 0 1 0, limit lower=-3.141592653589793 upper=3.141592653589793 effort=1e3 velocity=1e3
